File: uprom/23to27.brd (EAGLE design)
At the start: 26.7 x 39.4 mm, 10 parts, among them IC1 27C128P, T1 2N3904, T2 2N3904

Commit message: final boards
Parts:
- removed R1: (no value), rcl:0207/7
- removed R2, R3: (no value), rcl:R1206
- removed T1, T2: 2N3904, transistor-neu-to92:TO92
- removed TP2: TPSQTP16R, testpad:TP16R
Connections:
- removed net !SEL_E: R2.1, TP2.TP
- removed net !SEL_F_C: R1.1, SV1.8
- removed net N$1: R1.2, T1.2
- removed net N$2: R2.2, T2.2
- removed net N$3: T1.3, T2.1
- net !CS: now also SV1.8; no longer R3.2, T2.3
- net GND: no longer R3.1
- net VCC: no longer T1.1
Routing:
- net VCC: track 48.8 -> 22.9 mm
- net A11: track 27.6 -> 15.8 mm
- net !SEL_F_C: track 8.47 -> 0.00 mm
- net N$3: track 6.05 -> 0.00 mm
- net N$2: track 4.38 -> 0.00 mm
- net N$1: track 3.81 -> 0.00 mm
- net !CS: track 14.6 -> 11.4 mm
- net A12: track 18.0 -> 20.7 mm
