File: uprom/uprom2.sch (EAGLE design)
At the start: 6 parts, among them IC1 27C128P, IC2 74AC00D

Commit message: final boards
Parts:
- removed TP1, TP2: TPSQTP16R, testpad:TPSQTP16R
- added PAD1, PAD2: (no value), wirepad:1,6/0,8
- added R1: (no value), rcl:R-EU_R1206
Connections:
- removed net A13: IC1.A13, TP1.TP
- net !SEL_E: now also IC1.A13; no longer TP2.TP
- net GND: now also PAD1.P, PAD2.P, R1.1, R1.2
Other:
- moved on the sheet: IC2A, IC2B, IC2C, IC2D
